Commit message: fix(strafer_ros): wire sim-bridge topics through bringup
The Isaac Sim ROS 2 bridge publishes depth as `/d555/depth/*` and
stamps every topic with sim-time, neither of which matched the
real-robot pipeline the Jetson expected:

- timestamp_fixer: added a `restamp` parameter; when false the node
  becomes a pass-through relay so the bridge's sim-time stamps stay
  aligned with `/strafer/odom` (which does not go through the node).
  Defaults to true for real-robot use.
- bringup_sim_in_the_loop.launch.py: remap timestamp_fixer's depth
  inputs from `/d555/aligned_depth_to_color/*` to `/d555/depth/*`
  (sim camera is co-registered RGB+D so raw depth is already aligned),
  and set `restamp: false` so downstream sync works.
- strafer.urdf.xacro: add `d555_color_optical_frame` as a child of
  `d555_link`. The RealSense driver publishes this on hardware; the
  sim bridge does not, so carry it in the URDF for both modes.

File: source/strafer_ros/strafer_description/urdf/strafer.urdf.xacro (robot description, xacro)
@@ -210,3 +210,13 @@
     <origin xyz="${camera_x} ${camera_y} ${camera_z}" rpy="0 0 0"/>
   </joint>
+  <!-- Optical frame: camera convention (x=right, y=down, z=forward) rotated
+       from the physical d555_link (x=forward, y=left, z=up). The RealSense
+       driver publishes this on real hardware; the Isaac Sim bridge does not,
+       so carry it in the URDF so both modes have the same TF tree. -->
+  <link name="d555_color_optical_frame"/>
+  <joint name="d555_color_optical_joint" type="fixed">
+    <parent link="d555_link"/>
+    <child link="d555_color_optical_frame"/>
+    <origin xyz="0 0 0" rpy="${-pi/2} 0 ${-pi/2}"/>
+  </joint>
 </robot>
